Commit message: adding decimated meshes for gen3 lite arm and gripper

File: kortex_description/arms/gen3_lite/6dof/urdf/gen3_lite_macro.xacro (robot description, xacro)
@@ -22,5 +22,5 @@
         <origin xyz="0 0 0" rpy="0 0 0" />
         <geometry>
-          <mesh filename="package://kortex_description/arms/gen3_lite/${dof}dof/meshes/base_link.STL" />
+          <mesh filename="package://kortex_description/arms/gen3_lite/${dof}dof/meshes/base_link_decimated.stl" />
         </geometry>
       </collision>
@@ -47,5 +47,5 @@
         <origin xyz="0 0 0" rpy="0 0 0" />
         <geometry>
-          <mesh filename="package://kortex_description/arms/gen3_lite/${dof}dof/meshes/shoulder_link.STL" />
+          <mesh filename="package://kortex_description/arms/gen3_lite/${dof}dof/meshes/shoulder_link_decimated.stl" />
         </geometry>
       </collision>
@@ -79,5 +79,5 @@
         <origin xyz="0 0 0" rpy="0 0 0" />
         <geometry>
-          <mesh filename="package://kortex_description/arms/gen3_lite/${dof}dof/meshes/arm_link.STL" />
+          <mesh filename="package://kortex_description/arms/gen3_lite/${dof}dof/meshes/arm_link_decimated.stl" />
         </geometry>
       </collision>
@@ -111,5 +111,5 @@
         <origin xyz="0 0 0" rpy="0 0 0" />
         <geometry>
-          <mesh filename="package://kortex_description/arms/gen3_lite/${dof}dof/meshes/forearm_link.STL" />
+          <mesh filename="package://kortex_description/arms/gen3_lite/${dof}dof/meshes/forearm_link_decimated.stl" />
         </geometry>
       </collision>
@@ -143,5 +143,5 @@
         <origin xyz="0 0 0" rpy="0 0 0" />
         <geometry>
-          <mesh filename="package://kortex_description/arms/gen3_lite/${dof}dof/meshes/lower_wrist_link.STL" />
+          <mesh filename="package://kortex_description/arms/gen3_lite/${dof}dof/meshes/lower_wrist_link_decimated.stl" />
         </geometry>
       </collision>
@@ -175,5 +175,5 @@
         <origin xyz="0 0 0" rpy="0 0 0" />
         <geometry>
-          <mesh filename="package://kortex_description/arms/gen3_lite/${dof}dof/meshes/upper_wrist_link.STL" />
+          <mesh filename="package://kortex_description/arms/gen3_lite/${dof}dof/meshes/upper_wrist_link_decimated.stl" />
         </geometry>
       </collision>

File: kortex_description/grippers/gen3_lite_2f/urdf/gen3_lite_2f_macro.xacro (robot description, xacro)
@@ -35,5 +35,5 @@
         <origin xyz="0 0 0" rpy="0 0 0" />
         <geometry>
-          <mesh filename="package://kortex_description/grippers/gen3_lite_2f/meshes/gripper_base_link.STL" />
+          <mesh filename="package://kortex_description/grippers/gen3_lite_2f/meshes/gripper_base_link_decimated.stl" />
         </geometry>
       </collision>
@@ -60,5 +60,5 @@
       <origin xyz="0 0 0" rpy="0 0 0" />
       <geometry>
-        <mesh filename="package://kortex_description/grippers/gen3_lite_2f/meshes/right_finger_prox_link.STL" />
+        <mesh filename="package://kortex_description/grippers/gen3_lite_2f/meshes/right_finger_prox_link_decimated.stl" />
       </geometry>
     </collision>
@@ -92,5 +92,5 @@
         <origin xyz="0 0 0" rpy="0 0 0" />
         <geometry>
-          <mesh filename="package://kortex_description/grippers/gen3_lite_2f/meshes/right_finger_dist_link.STL" />
+          <mesh filename="package://kortex_description/grippers/gen3_lite_2f/meshes/right_finger_dist_link_decimated.stl" />
         </geometry>
       </collision>
@@ -125,5 +125,5 @@
         <origin xyz="0 0 0" rpy="0 0 0" />
         <geometry>
-          <mesh filename="package://kortex_description/grippers/gen3_lite_2f/meshes/left_finger_prox_link.STL" />
+          <mesh filename="package://kortex_description/grippers/gen3_lite_2f/meshes/left_finger_prox_link_decimated.stl" />
         </geometry>
       </collision>
@@ -158,5 +158,5 @@
         <origin xyz="0 0 0" rpy="0 0 0" />
         <geometry>
-          <mesh filename="package://kortex_description/grippers/gen3_lite_2f/meshes/left_finger_dist_link.STL" />
+          <mesh filename="package://kortex_description/grippers/gen3_lite_2f/meshes/left_finger_dist_link_decimated.stl" />
         </geometry>
       </collision>

Commit message: split visual and collision meshes

File: kortex_description/arms/gen3_lite/6dof/urdf/gen3_lite_macro.xacro (robot description, xacro)
@@ -13,14 +13,14 @@
         <origin xyz="0 0 0" rpy="0 0 0" />
         <geometry>
-          <mesh filename="package://kortex_description/arms/gen3_lite/${dof}dof/meshes/base_link.STL" />
-        </geometry>
-        <material name="">
-          <color rgba="0.803 0.824 0.820 1" />
-        </material>
-      </visual>
-      <collision>
-        <origin xyz="0 0 0" rpy="0 0 0" />
-        <geometry>
-          <mesh filename="package://kortex_description/arms/gen3_lite/${dof}dof/meshes/base_link.STL" />
+          <mesh filename="package://kortex_description/arms/gen3_lite/${dof}dof/meshes/visual/base_link.STL" />
+        </geometry>
+        <material name="">
+          <color rgba="0.803 0.824 0.820 1" />
+        </material>
+      </visual>
+      <collision>
+        <origin xyz="0 0 0" rpy="0 0 0" />
+        <geometry>
+          <mesh filename="package://kortex_description/arms/gen3_lite/${dof}dof/meshes/collision/base_link.STL" />
         </geometry>
       </collision>
@@ -38,14 +38,14 @@
         <origin xyz="0 0 0" rpy="0 0 0" />
         <geometry>
-          <mesh filename="package://kortex_description/arms/gen3_lite/${dof}dof/meshes/shoulder_link.STL" />
-        </geometry>
-        <material name="">
-          <color rgba="0.803 0.824 0.820 1" />
-        </material>
-      </visual>
-      <collision>
-        <origin xyz="0 0 0" rpy="0 0 0" />
-        <geometry>
-          <mesh filename="package://kortex_description/arms/gen3_lite/${dof}dof/meshes/shoulder_link.STL" />
+          <mesh filename="package://kortex_description/arms/gen3_lite/${dof}dof/meshes/visual/shoulder_link.STL" />
+        </geometry>
+        <material name="">
+          <color rgba="0.803 0.824 0.820 1" />
+        </material>
+      </visual>
+      <collision>
+        <origin xyz="0 0 0" rpy="0 0 0" />
+        <geometry>
+          <mesh filename="package://kortex_description/arms/gen3_lite/${dof}dof/meshes/collision/shoulder_link.STL" />
         </geometry>
       </collision>
@@ -70,14 +70,14 @@
         <origin xyz="0 0 0" rpy="0 0 0" />
         <geometry>
-          <mesh filename="package://kortex_description/arms/gen3_lite/${dof}dof/meshes/arm_link.STL" />
-        </geometry>
-        <material name="">
-          <color rgba="0.803 0.824 0.820 1" />
-        </material>
-      </visual>
-      <collision>
-        <origin xyz="0 0 0" rpy="0 0 0" />
-        <geometry>
-          <mesh filename="package://kortex_description/arms/gen3_lite/${dof}dof/meshes/arm_link.STL" />
+          <mesh filename="package://kortex_description/arms/gen3_lite/${dof}dof/meshes/visual/arm_link.STL" />
+        </geometry>
+        <material name="">
+          <color rgba="0.803 0.824 0.820 1" />
+        </material>
+      </visual>
+      <collision>
+        <origin xyz="0 0 0" rpy="0 0 0" />
+        <geometry>
+          <mesh filename="package://kortex_description/arms/gen3_lite/${dof}dof/meshes/collision/arm_link.STL" />
         </geometry>
       </collision>
@@ -102,14 +102,14 @@
         <origin xyz="0 0 0" rpy="0 0 0" />
         <geometry>
-          <mesh filename="package://kortex_description/arms/gen3_lite/${dof}dof/meshes/forearm_link.STL" />
-        </geometry>
-        <material name="">
-          <color rgba="0.803 0.824 0.820 1" />
-        </material>
-      </visual>
-      <collision>
-        <origin xyz="0 0 0" rpy="0 0 0" />
-        <geometry>
-          <mesh filename="package://kortex_description/arms/gen3_lite/${dof}dof/meshes/forearm_link.STL" />
+          <mesh filename="package://kortex_description/arms/gen3_lite/${dof}dof/meshes/visual/forearm_link.STL" />
+        </geometry>
+        <material name="">
+          <color rgba="0.803 0.824 0.820 1" />
+        </material>
+      </visual>
+      <collision>
+        <origin xyz="0 0 0" rpy="0 0 0" />
+        <geometry>
+          <mesh filename="package://kortex_description/arms/gen3_lite/${dof}dof/meshes/collision/forearm_link.STL" />
         </geometry>
       </collision>
@@ -134,14 +134,14 @@
         <origin xyz="0 0 0" rpy="0 0 0" />
         <geometry>
-          <mesh filename="package://kortex_description/arms/gen3_lite/${dof}dof/meshes/lower_wrist_link.STL" />
-        </geometry>
-        <material name="">
-          <color rgba="0.803 0.824 0.820 1" />
-        </material>
-      </visual>
-      <collision>
-        <origin xyz="0 0 0" rpy="0 0 0" />
-        <geometry>
-          <mesh filename="package://kortex_description/arms/gen3_lite/${dof}dof/meshes/lower_wrist_link.STL" />
+          <mesh filename="package://kortex_description/arms/gen3_lite/${dof}dof/meshes/visual/lower_wrist_link.STL" />
+        </geometry>
+        <material name="">
+          <color rgba="0.803 0.824 0.820 1" />
+        </material>
+      </visual>
+      <collision>
+        <origin xyz="0 0 0" rpy="0 0 0" />
+        <geometry>
+          <mesh filename="package://kortex_description/arms/gen3_lite/${dof}dof/meshes/collision/lower_wrist_link.STL" />
         </geometry>
       </collision>
@@ -166,14 +166,14 @@
         <origin xyz="0 0 0" rpy="0 0 0" />
         <geometry>
-          <mesh filename="package://kortex_description/arms/gen3_lite/${dof}dof/meshes/upper_wrist_link.STL" />
-        </geometry>
-        <material name="">
-          <color rgba="0.803 0.824 0.820 1" />
-        </material>
-      </visual>
-      <collision>
-        <origin xyz="0 0 0" rpy="0 0 0" />
-        <geometry>
-          <mesh filename="package://kortex_description/arms/gen3_lite/${dof}dof/meshes/upper_wrist_link.STL" />
+          <mesh filename="package://kortex_description/arms/gen3_lite/${dof}dof/meshes/visual/upper_wrist_link.STL" />
+        </geometry>
+        <material name="">
+          <color rgba="0.803 0.824 0.820 1" />
+        </material>
+      </visual>
+      <collision>
+        <origin xyz="0 0 0" rpy="0 0 0" />
+        <geometry>
+          <mesh filename="package://kortex_description/arms/gen3_lite/${dof}dof/meshes/collision/upper_wrist_link.STL" />
         </geometry>
       </collision>

File: kortex_description/grippers/gen3_lite_2f/urdf/gen3_lite_2f_macro.xacro (robot description, xacro)
@@ -26,5 +26,5 @@
         <origin xyz="0 0 0" rpy="0 0 0" />
         <geometry>
-          <mesh filename="package://kortex_description/grippers/gen3_lite_2f/meshes/gripper_base_link.STL" />
+          <mesh filename="package://kortex_description/grippers/gen3_lite_2f/meshes/visual/gripper_base_link.STL" />
         </geometry>
         <material name="">
@@ -35,5 +35,5 @@
         <origin xyz="0 0 0" rpy="0 0 0" />
         <geometry>
-          <mesh filename="package://kortex_description/grippers/gen3_lite_2f/meshes/gripper_base_link.STL" />
+          <mesh filename="package://kortex_description/grippers/gen3_lite_2f/meshes/collision/gripper_base_link.STL" />
         </geometry>
       </collision>
@@ -51,5 +51,5 @@
       <origin xyz="0 0 0" rpy="0 0 0" />
       <geometry>
-        <mesh filename="package://kortex_description/grippers/gen3_lite_2f/meshes/right_finger_prox_link.STL" />
+        <mesh filename="package://kortex_description/grippers/gen3_lite_2f/meshes/collision/right_finger_prox_link.STL" />
       </geometry>
       <material name="">
@@ -60,5 +60,5 @@
       <origin xyz="0 0 0" rpy="0 0 0" />
       <geometry>
-        <mesh filename="package://kortex_description/grippers/gen3_lite_2f/meshes/right_finger_prox_link.STL" />
+        <mesh filename="package://kortex_description/grippers/gen3_lite_2f/meshes/collision/right_finger_prox_link.STL" />
       </geometry>
     </collision>
@@ -83,5 +83,5 @@
         <origin xyz="0 0 0" rpy="0 0 0" />
         <geometry>
-          <mesh filename="package://kortex_description/grippers/gen3_lite_2f/meshes/right_finger_dist_link.STL" />
+          <mesh filename="package://kortex_description/grippers/gen3_lite_2f/meshes/collision/right_finger_dist_link.STL" />
         </geometry>
         <material name="">
@@ -92,5 +92,5 @@
         <origin xyz="0 0 0" rpy="0 0 0" />
         <geometry>
-          <mesh filename="package://kortex_description/grippers/gen3_lite_2f/meshes/right_finger_dist_link.STL" />
+          <mesh filename="package://kortex_description/grippers/gen3_lite_2f/meshes/collision/right_finger_dist_link.STL" />
         </geometry>
       </collision>
@@ -116,5 +116,5 @@
         <origin xyz="0 0 0" rpy="0 0 0" />
         <geometry>
-          <mesh filename="package://kortex_description/grippers/gen3_lite_2f/meshes/left_finger_prox_link.STL" />
+          <mesh filename="package://kortex_description/grippers/gen3_lite_2f/meshes/collision/left_finger_prox_link.STL" />
         </geometry>
         <material name="">
@@ -125,5 +125,5 @@
         <origin xyz="0 0 0" rpy="0 0 0" />
         <geometry>
-          <mesh filename="package://kortex_description/grippers/gen3_lite_2f/meshes/left_finger_prox_link.STL" />
+          <mesh filename="package://kortex_description/grippers/gen3_lite_2f/meshes/collision/left_finger_prox_link.STL" />
         </geometry>
       </collision>
@@ -149,5 +149,5 @@
         <origin xyz="0 0 0" rpy="0 0 0" />
         <geometry>
-          <mesh filename="package://kortex_description/grippers/gen3_lite_2f/meshes/left_finger_dist_link.STL" />
+          <mesh filename="package://kortex_description/grippers/gen3_lite_2f/meshes/collision/left_finger_dist_link.STL" />
         </geometry>
         <material name="">
@@ -158,5 +158,5 @@
         <origin xyz="0 0 0" rpy="0 0 0" />
         <geometry>
-          <mesh filename="package://kortex_description/grippers/gen3_lite_2f/meshes/left_finger_dist_link.STL" />
+          <mesh filename="package://kortex_description/grippers/gen3_lite_2f/meshes/collision/left_finger_dist_link.STL" />
         </geometry>
       </collision>
